File: STHDAQ_BX/STHDAQ_BX.kicad_pcb (KiCad board)
At the start: 2 copper layers, 36 x 56 mm, 48 parts, among them J1 532611071, P1 S2B-PH-SM4-TB, U1 ADS1256IDBR, U2 ADP151AUJZ-3.0-R7, U3 OPA350UA, U4 REF5025AIDR, U5 102010448, U6 LT1461AIS8-5-PBF, Y1 ABLS-8MHZ-K4T

Commit message: BX pcb layouting
Parts:
- added H1: MountingHole, MountingHole:MountingHole_3.2mm_M3_ISO14580_Pad_TopBottom, F.Cu at (201.9, 84.1)
- added H2: MountingHole, MountingHole:MountingHole_3.2mm_M3_ISO14580_Pad_TopBottom, F.Cu at (174.0, 84.2)
- added H3: MountingHole, MountingHole:MountingHole_3.2mm_M3_ISO14580_Pad_TopBottom, F.Cu at (174.0, 132.0)
- added H4: MountingHole, MountingHole:MountingHole_3.2mm_M3_ISO14580_Pad_TopBottom, F.Cu at (201.9, 131.9)
- P1: footprint daFootprints:JST_S2B-PH-SM4-TB -> daFootprintsBX:JST_S2B-PH-SM4-TB
- U6: footprint daFootprints:SOIC127P600X175-8N -> daFootprintsBX:SOIC127P600X175-8N
- moved C1 60.3 mm to (203.3, 121.4), turned to 180 degrees
- moved C2 58.2 mm to (198.9, 125.5), turned to 180 degrees
- moved C10 55.5 mm to (196.8, 127.1), turned to 180 degrees
- moved C11 53.7 mm to (196.8, 126.1), turned to 180 degrees
- moved C9 41.0 mm to (185.4, 116.3)
- moved C8 35.4 mm to (185.4, 115.1)
- moved R2 35.2 mm to (188.2, 110.8), turned to 90 degrees
- moved R16 31.3 mm to (193.3, 110.9), turned to -90 degrees
- moved R11 30.7 mm to (186.5, 110.8), turned to 90 degrees
- moved R15 30.7 mm to (191.7, 110.9), turned to -90 degrees
- moved R14 30.0 mm to (189.9, 110.8), turned to -90 degrees
- moved R12 28.1 mm to (184.5, 110.8), turned to 90 degrees
- moved R13 25.6 mm to (182.8, 110.8), turned to 90 degrees
- moved C13 7.84 mm to (196.3, 125.0), turned to 180 degrees
- moved C12 5.99 mm to (196.3, 124.2), turned to 180 degrees
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Routing:
- net 5BVCC: track 0.00 -> 49.1 mm, vias 0 -> 4
- net Net-(U5-A3/D3): track 0.00 -> 27.0 mm, vias 0 -> 2
- net Net-(U5-A2/D2): track 0.00 -> 26.5 mm, vias 0 -> 2
- net Net-(U5-A1/D1): track 0.00 -> 26.3 mm, vias 0 -> 2
- net Net-(U5-A0/D0): track 0.00 -> 25.7 mm, vias 0 -> 2
- net REF2.5: track 0.00 -> 25.5 mm, vias 0 -> 2
- net /RESET: track 0.00 -> 23.1 mm, vias 0 -> 2
- net /SYNC/PDWN: track 0.00 -> 20.8 mm, vias 0 -> 2
- net /CS: track 0.00 -> 16.4 mm
- net /XTAL1: track 0.00 -> 16.2 mm
- net /DRDY: track 0.00 -> 14.9 mm
- net /SCLK: track 0.00 -> 13.6 mm, vias 0 -> 2
- net /S1+: track 0.00 -> 13.3 mm
- net /DOUT: track 0.00 -> 12.8 mm
- net /S1-: track 0.00 -> 12.7 mm
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- added copper zone on F.Cu, net 5VCC
- added copper zone on B.Cu, net Earth
Other:
- outline, holes or cut-outs redrawn
