File: STHDAQ_BX/STHDAQ_BX.kicad_sch (KiCad schematic)
At the start: 48 parts, among them J1 532611071, P1 S2B-PH-SM4-TB, U1 ADS1256IDBR, U2 ADP151AUJZ-3.0-R7, U3 OPA350UA, U4 REF5025AIDR, U5 102010448, U6 LT1461AIS8-5-PBF, Y1 ABLS-8MHZ-K4T

Commit message: BX pcb layouting
Parts:
- added H1, H2, H3, H4: MountingHole, MountingHole:MountingHole_3.2mm_M3_ISO14580_Pad_TopBottom, symbol Mechanical:MountingHole
- P1: footprint daFootprints:JST_S2B-PH-SM4-TB -> daFootprintsBX:JST_S2B-PH-SM4-TB
- U6: footprint daFootprints:SOIC127P600X175-8N -> daFootprintsBX:SOIC127P600X175-8N

Commit message: Changes in BX
Parts:
- removed C22: 1u, Capacitor_SMD:C_0201_0603Metric_Pad0.64x0.40mm_HandSolder, symbol Device:C
- removed U6: LT1461AIS8-5-PBF, daFootprintsBX:SOIC127P600X175-8N, symbol LT1461AIS8-5_PBF:LT1461AIS8-5-PBF
- C1, C10, C11, C12, C13, C14, C15, C16, C17, C18, C19, C2, C20, C21, C23, C3, C4, C5, C6, C7, C8, C9: footprint Capacitor_SMD:C_0201_0603Metric_Pad0.64x0.40mm_HandSolder -> Capacitor_SMD:C_0603_1608Metric_Pad1.08x0.95mm_HandSolder
- R1, R10, R11, R12, R13, R14, R15, R16, R2, R3, R4, R5, R6, R7, R8, R9: footprint Resistor_SMD:R_0201_0603Metric_Pad0.64x0.40mm_HandSolder -> Resistor_SMD:R_0603_1608Metric_Pad0.98x0.95mm_HandSolder
Connections:
- net 5VCC is gone; now on net 5BVCC: C1.2, C3.2, C7.2, C8.2, C9.2, P1.1, U1.1 (AVDD), U2.1 (VIN), U2.3 (EN), U3.7 (V+), U4.2 (VIN), U5.VUSB
- no-connect marks 26 -> 25
